Commit message: Add mapper_params

File: description/core.xacro (robot description, xacro)
@@ -1,6 +1,47 @@
 <?xml version="1.0"?>
-<robot xmlns:xacro="http://www.ros.org/wiki/xacro">
-<!-- Базовая ссылка -->
+<robot xmlns:xacro="http://www.ros.org/wiki/xacro" >
+    <xacro:property name="chassis_length" value="0.200"/>
+    <xacro:property name="chassis_width" value="0.160"/>
+    <xacro:property name="chassis_height" value="0.050"/>
+    <xacro:property name="chassis_mass" value="1.0"/>
+    <xacro:property name="chassis_offset_x" value="-0.06"/>
+    <xacro:property name="chassis_offset_y" value="0"/>
+    <xacro:property name="chassis_offset_z" value="0.095"/>
+    <xacro:property name="wheel_radius" value="0.035"/>
+    <xacro:property name="wheel_thickness" value="0.020"/>
+    <xacro:property name="wheel_mass" value="0.05"/>
+    <xacro:property name="wheel_offset_x" value="0.226"/>
+    <xacro:property name="wheel_offset_y" value="0.035"/>
+    <xacro:property name="wheel_offset_z" value="0.01"/>
+    <xacro:property name="caster_wheel_radius" value="0.02"/>
+    <xacro:property name="caster_wheel_mass" value="0.5"/>
+    <xacro:property name="caster_wheel_offset_x" value="0.12"/>
+    <xacro:property name="caster_wheel_offset_y" value="0.03"/>
+    <xacro:property name="caster_wheel_offset_z" value="0.015"/>
+    <material name="white">
+        <color rgba="1 1 1 1" />
+    </material>
+    <material name="orange">
+        <color rgba="1 0.3 0.1 1"/>
+    </material>
+    <material name="blue">
+        <color rgba="0.2 0.2 1 1"/>
+    </material>
+    <material name="black">
+        <color rgba="0 0 0 1"/>
+    </material>
+    <material name="red">
+        <color rgba="1 0 0 1"/>
+    </material>
+    <!-- Базовая ссылка -->
     <link name="base_link">
+    </link>
+    <!-- След базовой ссылки -->
+    <joint name="base_footprint_joint" type="fixed">
+        <parent link="base_link"/>
+        <child link="base_footprint"/>
+        <origin xyz="0 0 0" rpy="0 0 0"/>
+    </joint>
+    <link name="base_footprint">
     </link>
     <!-- Шасси -->
@@ -8,13 +49,20 @@
         <parent link="base_link"/>
         <child link="chassis"/>
-        <origin xyz="0 0 0"/>
+        <origin xyz="${chassis_offset_x} ${chassis_offset_y} ${chassis_offset_z}"/>
     </joint>
     <link name="chassis">
         <visual>
-            <origin xyz="0 0 0.035"/>
+            <origin xyz="0 0 0"/>
             <geometry>
-                <cylinder radius="0.17" length="0.07"/>
+                <box size="${chassis_length} ${chassis_width} ${chassis_height}"/>
             </geometry>
+            <material name="orange"/>
         </visual>
+        <collision>
+            <origin xyz="${chassis_length/2} 0 ${chassis_height/2}"/>
+            <geometry>
+                <box size="${chassis_length} ${chassis_width} ${chassis_height}"/>
+            </geometry>
+        </collision>
     </link>
     <!-- Левое колесо -->
@@ -22,14 +70,19 @@
         <parent link="base_link"/>
         <child link="left_wheel"/>
-        <origin xyz="0 0.115 0"/>
-        <axis xyz="0 1 0"/>
+        <origin xyz="0 ${wheel_offset_y} 0" rpy="-${pi/2} 0 0" />
+        <axis xyz="0 0 1"/>
     </joint>
     <link name="left_wheel">
         <visual>
-            <origin xyz="0 0 0" rpy="${pi/2} 0 0"/>
             <geometry>
-                <cylinder radius="0.035" length="0.02"/>
+                <cylinder radius="${wheel_radius}" length="${wheel_thickness}"/>
             </geometry>
+            <material name="blue"/>
         </visual>
+        <collision>
+            <geometry>
+                <sphere radius="${wheel_radius}"/>
+            </geometry>
+        </collision>
     </link>
     <!-- Правое колесо -->
@@ -37,27 +90,57 @@
         <parent link="base_link"/>
         <child link="right_wheel"/>
-        <origin xyz="0 -0.115 0"/>
-        <axis xyz="0 1 0"/>
+        <origin xyz="0 ${-wheel_offset_y} 0" rpy="${pi/2} 0 0" />
+        <axis xyz="0 0 -1"/>
     </joint>
     <link name="right_wheel">
         <visual>
-            <origin xyz="0 0 0" rpy="${pi/2} 0 0"/>
             <geometry>
-                <cylinder radius="0.035" length="0.02"/>
+                <cylinder radius="${wheel_radius}" length="${wheel_thickness}"/>
             </geometry>
+            <material name="blue"/>
         </visual>
+        <collision>
+            <geometry>
+                <sphere radius="${wheel_radius}"/>
+            </geometry>
+        </collision>
     </link>
-    <!-- Переднее колесо -->
-    <joint name="caster_wheel_joint" type="fixed">
-        <parent link="chassis"/>
-        <child link="caster_wheel"/>
-        <origin xyz="0.115 0 0"/>
+    <!-- Левое поддерживающее колесо -->
+    <joint name="left_caster_wheel_joint" type="fixed">
+        <parent link="base_link"/>
+        <child link="left_caster_wheel"/>
+        <origin xyz="${-caster_wheel_offset_x} ${caster_wheel_offset_y} ${-caster_wheel_offset_z}"/>
     </joint>
-    <link name="caster_wheel">
+    <link name="left_caster_wheel">
         <visual>
             <geometry>
-                <sphere radius="0.035"/>
+                <sphere radius="${caster_wheel_radius}"/>
             </geometry>
+            <material name="white"/>
         </visual>
+        <collision>
+            <geometry>
+                <sphere radius="${caster_wheel_radius}"/>
+            </geometry>
+        </collision>
+    </link>
+    <!-- Правое поддерживающее колесо -->
+    <joint name="right_caster_wheel_joint" type="fixed">
+        <parent link="base_link"/>
+        <child link="right_caster_wheel"/>
+        <origin xyz="${-caster_wheel_offset_x} ${-caster_wheel_offset_y} ${-caster_wheel_offset_z}"/>
+    </joint>
+    <link name="right_caster_wheel">
+        <visual>
+            <geometry>
+                <sphere radius="${caster_wheel_radius}"/>
+            </geometry>
+            <material name="white"/>
+        </visual>
+        <collision>
+            <geometry>
+                <sphere radius="${caster_wheel_radius}"/>
+            </geometry>
+        </collision>
     </link>
 </robot>
